Commit message: changes to work with rmf_sim launch

File: rotors_description/urdf/delta_collision_check_base.xacro (robot description, xacro)
@@ -19,5 +19,5 @@
   <xacro:include filename="$(find rotors_description)/urdf/component_snippets.xacro" />
   <!-- Instantiate firefly "mechanics" -->
-  <xacro:include filename="$(find rotors_description)/urdf/rmf_obelix.xacro" />
+  <xacro:include filename="$(find rotors_description)/urdf/rmf_obelix_bigger.xacro" />
   <!-- Instantiate a controller. -->
   <xacro:controller_plugin_macro namespace="${namespace}" imu_sub_topic="imu" />
@@ -41,8 +41,3 @@
       wait_to_record_bag="$(arg wait_to_record_bag)" />
   </xacro:if>
-  <!-- Add an 0S0-128 lidar -->
-  <xacro:include filename="$(find lidar_description)/urdf/OS0-128.urdf.xacro"/>
-  <xacro:OS0-128 parent="${namespace}/base_link" name="${namespace}/velodyne" topic="velodyne_points" hz="10" lasers="64" samples="440" collision_range="0.3" min_range="0.3" max_range="50.0">
-    <origin xyz="0 0 0.04" rpy="0 0 0" />
-  </xacro:OS0-128>
 </robot>
